File: Hardware/PCB/Projet_Controler V3 - Copie/Projet_Controler.kicad_sch (KiCad schematic)
At the start: 4 parts

Commit message: update pcb
Parts:
- removed H1, H2, H3, H4: MountingHole, symbol Mechanical:MountingHole
- added H101, H102, H103, H104: MountingHole_Pad, MountingHole:MountingHole_2.7mm_M2.5_DIN965_Pad, symbol Mechanical:MountingHole_Pad
Connections:
- new net GND: H101.1, H102.1, H103.1, H104.1
Other:
- sheet BLUETOOTH ports: added KEY; removed none
- sheet STM32 ports: added KEY; removed TOF_PWR_EN, USART2_RX, USART2_TX
