File: Hardware/PCB/Projet_Controler V3 - Copie/bluetooth.kicad_sch (KiCad schematic)
At the start: 1 part, among them U4 HC-05

Commit message: update pcb
Parts:
- added D501, D502: LED, LED_SMD:LED_0603_1608Metric, symbol Device:LED
- added R501, R502: 820, Resistor_SMD:R_0402_1005Metric, symbol Device:R_Small
- renumbered U4 to U501
Connections:
- net GND: now also D501.1 (K), D502.1 (K)
- net LED_1: now reaches U501.31 (PIO[8])
- net LED_1: now also R501.1
- net LED_2: now reaches U501.32 (PIO[9])
- net LED_2: now also R502.1
- net KEY: now reaches U501.34 (PIO[11])
- new net: D502.2 (A), R502.2
- new net: D501.2 (A), R501.2
- no-connect marks 27 -> 24
Other:
- note added: "LED, 2mA @ 1.7V"
Changed lines of the file:
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@@
   (no_connect (at 166.37 66.04))
   (no_connect (at 166.37 86.36))
-  (no_connect (at 166.37 83.82))
   (no_connect (at 125.73 68.58))
   (no_connect (at 166.37 78.74))
-  (no_connect (at 166.37 81.28))
-  (no_connect (at 166.37 88.9))
   (no_connect (at 166.37 96.52))
   (no_connect (at 166.37 63.5))
@@
     (stroke (width 0) (type default))
   )
-  (polyline (pts (xy 189.23 44.45) (xy 189.23 120.65))
-    (stroke (width 0) (type default))
-  )
-  (polyline (pts (xy 101.6 44.45) (xy 189.23 44.45))
+  (wire (pts (xy 204.47 80.01) (xy 204.47 82.55))
+    (stroke (width 0) (type default))
+  )
+  (polyline (pts (xy 233.68 44.45) (xy 233.68 120.65))
+    (stroke (width 0) (type default))
+  )
+  (polyline (pts (xy 101.6 44.45) (xy 233.68 44.45))
     (stroke (width 0) (type default))
   )
@@
     (stroke (width 0) (type default))
   )
-  (polyline (pts (xy 189.23 120.65) (xy 101.6 120.65))
+  (polyline (pts (xy 233.68 120.65) (xy 101.6 120.65))
+    (stroke (width 0) (type default))
+  )
+  (wire (pts (xy 217.17 80.01) (xy 217.17 82.55))
+    (stroke (width 0) (type default))
+  )
+  (wire (pts (xy 204.47 59.69) (xy 204.47 66.04))
+    (stroke (width 0) (type default))
+  )
+  (wire (pts (xy 166.37 81.28) (xy 177.8 81.28))
+    (stroke (width 0) (type default))
+  )
+  (wire (pts (xy 217.17 71.12) (xy 217.17 72.39))
+    (stroke (width 0) (type default))
+  )
+  (wire (pts (xy 166.37 83.82) (xy 177.8 83.82))
     (stroke (width 0) (type default))
   )
@@
     (stroke (width 0) (type default))
   )
+  (wire (pts (xy 217.17 59.69) (xy 217.17 66.04))
+    (stroke (width 0) (type default))
+  )
   (polyline (pts (xy 101.6 44.45) (xy 101.6 120.65))
     (stroke (width 0) (type default))
   )
+  (wire (pts (xy 204.47 71.12) (xy 204.47 72.39))
+    (stroke (width 0) (type default))
+  )
   (wire (pts (xy 168.91 55.88) (xy 166.37 55.88))
     (stroke (width 0) (type default))
+  )
+  (text "LED, 2mA @ 1.7V" (at 214.63 48.26 0)
+    (effects (font (size 1.27 1.27)) (justify left bottom))
   )
   (text "Module HC-05" (at 102.87 48.26 0)
     (effects (font (size 1.27 1.27)) (justify left bottom))
   )
+  (label "LED_2" (at 217.17 59.69 270) (fields_autoplaced)
+    (effects (font (size 1.27 1.27)) (justify right bottom))
+  )
+  (label "LED_2" (at 177.8 83.82 180) (fields_autoplaced)
+    (effects (font (size 1.27 1.27)) (justify right bottom))
+  )
+  (label "LED_1" (at 204.47 59.69 270) (fields_autoplaced)
+    (effects (font (size 1.27 1.27)) (justify right bottom))
+  )
+  (label "LED_1" (at 177.8 81.28 180) (fields_autoplaced)
+    (effects (font (size 1.27 1.27)) (justify right bottom))
+  )
   (hierarchical_label "USART1_TX" (shape output) (at 125.73 71.12 180) (fields_autoplaced)
     (effects (font (size 1.27 1.27)) (justify right))
@@
     (effects (font (size 1.27 1.27)) (justify right))
   )
+  (hierarchical_label "KEY" (shape input) (at 166.37 88.9 0) (fields_autoplaced)
+    (effects (font (size 1.27 1.27)) (justify left))
+  )
   (symbol (lib_id "HC-05:HC-05") (at 146.05 83.82 0) (unit 1)
     (in_bom yes) (on_board yes) (dnp no) (fields_autoplaced)
-    (property "Reference" "U4" (at 146.05 49.53 0)
+    (property "Reference" "U501" (at 146.05 49.53 0)
       (effects (font (size 1.27 1.27)))
     )
@@
       (project "Projet_Controler"
         (path "/3b08c5cd-ddb4-4590-8a64-446919e151a7/8bd56d3a-8f5f-47c9-8667-6b19a6154c75"
-          (reference "U4") (unit 1)
+          (reference "U501") (unit 1)
+        )
+      )
+    )
+  )
+  (symbol (lib_id "Device:R_Small") (at 217.17 68.58 0) (unit 1)
+    (in_bom yes) (on_board yes) (dnp no) (fields_autoplaced)
+    (property "Reference" "R502" (at 219.71 67.31 0)
+      (effects (font (size 1.27 1.27)) (justify left))
+    )
+    (property "Value" "820" (at 219.71 69.85 0)
+      (effects (font (size 1.27 1.27)) (justify left))
+    )
+    (property "Footprint" "Resistor_SMD:R_0402_1005Metric" (at 217.17 68.58 0)
+      (effects (font (size 1.27 1.27)) hide)
+    )
+    (property "Datasheet" "~" (at 217.17 68.58 0)
+      (effects (font (size 1.27 1.27)) hide)
+    )
+    (pin "1")
+    (pin "2")
+    (instances
+      (project "Projet_Controler"
+        (path "/3b08c5cd-ddb4-4590-8a64-446919e151a7/8bd56d3a-8f5f-47c9-8667-6b19a6154c75"
+          (reference "R502") (unit 1)
         )
       )
@@
   (symbol (lib_id "power:GND") (at 168.91 110.49 0) (unit 1)
     (in_bom yes) (on_board yes) (dnp no) (fields_autoplaced)
-    (property "Reference" "#PWR029" (at 168.91 116.84 0)
+    (property "Reference" "#PWR0502" (at 168.91 116.84 0)
       (effects (font (size 1.27 1.27)) hide)
     )
@@
       (project "Projet_Controler"
         (path "/3b08c5cd-ddb4-4590-8a64-446919e151a7/8bd56d3a-8f5f-47c9-8667-6b19a6154c75"
-          (reference "#PWR029") (unit 1)
+          (reference "#PWR0502") (unit 1)
         )
       )
@@
   (symbol (lib_id "power:+3.3V") (at 168.91 54.61 0) (unit 1)
     (in_bom yes) (on_board yes) (dnp no) (fields_autoplaced)
-    (property "Reference" "#PWR028" (at 168.91 58.42 0)
+    (property "Reference" "#PWR0501" (at 168.91 58.42 0)
       (effects (font (size 1.27 1.27)) hide)
     )
@@
       (project "Projet_Controler"
         (path "/3b08c5cd-ddb4-4590-8a64-446919e151a7/8bd56d3a-8f5f-47c9-8667-6b19a6154c75"
-          (reference "#PWR028") (unit 1)
-        )
-      )
+          (reference "#PWR0501") (unit 1)
+        )
+      )
+    )
+  )
+  (symbol (lib_id "Device:LED") (at 217.17 76.2 90) (unit 1)
+    (in_bom yes) (on_board yes) (dnp no) (fields_autoplaced)
+    (property "Reference" "D502" (at 220.98 76.5175 90)
+      (effects (font (size 1.27 1.27)) (justify right))
+    )
+    (property "Value" "LED" (at 220.98 79.0575 90)
+      (effects (font (size 1.27 1.27)) (justify right))
+    )
+    (property "Footprint" "LED_SMD:LED_0603_1608Metric" (at 217.17 76.2 0)
+      (effects (font (size 1.27 1.27)) hide)
+    )
+    (property "Datasheet" "~" (at 217.17 76.2 0)
+      (effects (font (size 1.27 1.27)) hide)
+    )
+    (pin "2")
+    (pin "1")
+    (instances
+      (project "Projet_Controler"
+        (path "/3b08c5cd-ddb4-4590-8a64-446919e151a7/8bd56d3a-8f5f-47c9-8667-6b19a6154c75"
+          (reference "D502") (unit 1)
+        )
+      )
+    )
+  )
+  (symbol (lib_id "power:GND") (at 204.47 82.55 0) (unit 1)
+    (in_bom yes) (on_board yes) (dnp no) (fields_autoplaced)
+    (property "Reference" "#PWR0503" (at 204.47 88.9 0)
+      (effects (font (size 1.27 1.27)) hide)
+    )
+    (property "Value" "GND" (at 204.47 87.63 0)
+      (effects (font (size 1.27 1.27)))
+    )
+    (property "Footprint" "" (at 204.47 82.55 0)
+      (effects (font (size 1.27 1.27)) hide)
+    )
+    (property "Datasheet" "" (at 204.47 82.55 0)
+      (effects (font (size 1.27 1.27)) hide)
+    )
+    (pin "1")
+    (instances
+      (project "Projet_Controler"
+        (path "/3b08c5cd-ddb4-4590-8a64-446919e151a7/8bd56d3a-8f5f-47c9-8667-6b19a6154c75"
+          (reference "#PWR0503") (unit 1)
+        )
+      )
+    )
+  )
+  (symbol (lib_id "Device:LED") (at 204.47 76.2 90) (unit 1)
+    (in_bom yes) (on_board yes) (dnp no) (fields_autoplaced)
+    (property "Reference" "D501" (at 208.28 76.5175 90)
+      (effects (font (size 1.27 1.27)) (justify right))
+    )
+    (property "Value" "LED" (at 208.28 79.0575 90)
+      (effects (font (size 1.27 1.27)) (justify right))
+    )
+    (property "Footprint" "LED_SMD:LED_0603_1608Metric" (at 204.47 76.2 0)
+      (effects (font (size 1.27 1.27)) hide)
+    )
+    (property "Datasheet" "~" (at 204.47 76.2 0)
+      (effects (font (size 1.27 1.27)) hide)
+    )
+    (pin "2")
+    (pin "1")
+    (instances
+      (project "Projet_Controler"
+        (path "/3b08c5cd-ddb4-4590-8a64-446919e151a7/8bd56d3a-8f5f-47c9-8667-6b19a6154c75"
+          (reference "D501") (unit 1)
+        )
+      )
+    )
+  )
+  (symbol (lib_id "power:GND") (at 217.17 82.55 0) (unit 1)
+    (in_bom yes) (on_board yes) (dnp no) (fields_autoplaced)
+    (property "Reference" "#PWR0504" (at 217.17 88.9 0)
+      (effects (font (size 1.27 1.27)) hide)
+    )
+    (property "Value" "GND" (at 217.17 87.63 0)
+      (effects (font (size 1.27 1.27)))
+    )
+    (property "Footprint" "" (at 217.17 82.55 0)
+      (effects (font (size 1.27 1.27)) hide)
+    )
+    (property "Datasheet" "" (at 217.17 82.55 0)
+      (effects (font (size 1.27 1.27)) hide)
+    )
+    (pin "1")
+    (instances
+      (project "Projet_Controler"
+        (path "/3b08c5cd-ddb4-4590-8a64-446919e151a7/8bd56d3a-8f5f-47c9-8667-6b19a6154c75"
+          (reference "#PWR0504") (unit 1)
+        )
+      )
+    )
+  )
+  (symbol (lib_id "Device:R_Small") (at 204.47 68.58 0) (unit 1)
+    (in_bom yes) (on_board yes) (dnp no) (fields_autoplaced)
+    (property "Reference" "R501" (at 207.01 67.31 0)
+      (effects (font (size 1.27 1.27)) (justify left))
+    )
+    (property "Value" "820" (at 207.01 69.85 0)
+      (effects (font (size 1.27 1.27)) (justify left))
+    )
+    (property "Footprint" "Resistor_SMD:R_0402_1005Metric" (at 204.47 68.58 0)
+      (effects (font (size 1.27 1.27)) hide)
+    )
+    (property "Datasheet" "~" (at 204.47 68.58 0)
+      (effects (font (size 1.27 1.27)) hide)
+    )
+    (pin "1")
+    (pin "2")
+    (instances
+      (project "Projet_Controler"
+        (path "/3b08c5cd-ddb4-4590-8a64-446919e151a7/8bd56d3a-8f5f-47c9-8667-6b19a6154c75"
+          (reference "R501") (unit 1)
+        )
+      )
