File: Hardware/PCB/Projet_Controler V3 - Copie/motor.kicad_sch (KiCad schematic)
At the start: 5 parts, among them J3 Conn_01x02, Q1 SQ2310ES-T1

Commit message: update pcb
Parts:
- D601: renamed from D1; footprint DIOM7959X262N -> mod:DIOM7959X262N
- J601: renamed from J3; footprint (none) -> Connector_PinHeader_1.27mm:PinHeader_1x02_P1.27mm_Vertical
- Q601: renamed from Q1; footprint SOT95P237X112-3N -> mod:SOT95P237X112-3N
- R601: renamed from R11; footprint (none) -> Resistor_SMD:R_0402_1005Metric
- R602: renamed from R12; footprint (none) -> Resistor_SMD:R_0402_1005Metric
Connections:
- net drain ?: no longer names the net of D601.2 (A), J601.2 (Pin_2), Q601.3 (D)
Changed lines of the file:
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@@
     (effects (font (size 1.27 1.27)) (justify left bottom))
-  )
-  (global_label "drain ?" (shape input) (at 154.94 86.36 180) (fields_autoplaced)
-    (effects (font (size 1.27 1.27)) (justify right))
-    (property "Intersheetrefs" "${INTERSHEET_REFS}" (at 145.3456 86.36 0)
-      (effects (font (size 1.27 1.27)) (justify right) hide)
-    )
   )
   (hierarchical_label "PWM" (shape input) (at 142.24 99.06 180) (fields_autoplaced)
@@
   (symbol (lib_id "power:+3.3V") (at 162.56 67.31 0) (unit 1)
     (in_bom yes) (on_board yes) (dnp no) (fields_autoplaced)
-    (property "Reference" "#PWR019" (at 162.56 71.12 0)
+    (property "Reference" "#PWR0601" (at 162.56 71.12 0)
       (effects (font (size 1.27 1.27)) hide)
     )
@@
       (project "Projet_Controler"
         (path "/3b08c5cd-ddb4-4590-8a64-446919e151a7/d5df5f48-8d85-45ba-9c59-31e00cd39d16"
-          (reference "#PWR019") (unit 1)
+          (reference "#PWR0601") (unit 1)
         )
       )
@@
   (symbol (lib_id "Device:R_Small_US") (at 144.78 99.06 90) (unit 1)
     (in_bom yes) (on_board yes) (dnp no) (fields_autoplaced)
-    (property "Reference" "R11" (at 144.78 93.98 90)
+    (property "Reference" "R601" (at 144.78 93.98 90)
       (effects (font (size 1.27 1.27)))
     )
@@
       (effects (font (size 1.27 1.27)))
     )
-    (property "Footprint" "" (at 144.78 99.06 0)
+    (property "Footprint" "Resistor_SMD:R_0402_1005Metric" (at 144.78 99.06 0)
       (effects (font (size 1.27 1.27)) hide)
     )
@@
       (project "Projet_Controler"
         (path "/3b08c5cd-ddb4-4590-8a64-446919e151a7/d5df5f48-8d85-45ba-9c59-31e00cd39d16"
-          (reference "R11") (unit 1)
+          (reference "R601") (unit 1)
         )
       )
@@
   (symbol (lib_id "Device:R_Small_US") (at 149.86 104.14 0) (unit 1)
     (in_bom yes) (on_board yes) (dnp no) (fields_autoplaced)
-    (property "Reference" "R12" (at 152.4 103.505 0)
+    (property "Reference" "R602" (at 152.4 103.505 0)
       (effects (font (size 1.27 1.27)) (justify left))
     )
@@
       (effects (font (size 1.27 1.27)) (justify left))
     )
-    (property "Footprint" "" (at 149.86 104.14 0)
+    (property "Footprint" "Resistor_SMD:R_0402_1005Metric" (at 149.86 104.14 0)
       (effects (font (size 1.27 1.27)) hide)
     )
@@
       (project "Projet_Controler"
         (path "/3b08c5cd-ddb4-4590-8a64-446919e151a7/d5df5f48-8d85-45ba-9c59-31e00cd39d16"
-          (reference "R12") (unit 1)
+          (reference "R602") (unit 1)
         )
       )
@@
   (symbol (lib_id "Connector_Generic:Conn_01x02") (at 172.72 83.82 0) (unit 1)
     (in_bom yes) (on_board yes) (dnp no) (fields_autoplaced)
-    (property "Reference" "J3" (at 175.26 84.455 0)
+    (property "Reference" "J601" (at 175.26 84.455 0)
       (effects (font (size 1.27 1.27)) (justify left))
     )
@@
       (effects (font (size 1.27 1.27)) (justify left))
     )
-    (property "Footprint" "" (at 172.72 83.82 0)
+    (property "Footprint" "Connector_PinHeader_1.27mm:PinHeader_1x02_P1.27mm_Vertical" (at 172.72 83.82 0)
       (effects (font (size 1.27 1.27)) hide)
     )
@@
       (project "Projet_Controler"
         (path "/3b08c5cd-ddb4-4590-8a64-446919e151a7/d5df5f48-8d85-45ba-9c59-31e00cd39d16"
-          (reference "J3") (unit 1)
+          (reference "J601") (unit 1)
         )
       )
@@
   (symbol (lib_id "power:GND") (at 162.56 114.3 0) (unit 1)
     (in_bom yes) (on_board yes) (dnp no) (fields_autoplaced)
-    (property "Reference" "#PWR020" (at 162.56 120.65 0)
+    (property "Reference" "#PWR0602" (at 162.56 120.65 0)
       (effects (font (size 1.27 1.27)) hide)
     )
@@
       (project "Projet_Controler"
         (path "/3b08c5cd-ddb4-4590-8a64-446919e151a7/d5df5f48-8d85-45ba-9c59-31e00cd39d16"
-          (reference "#PWR020") (unit 1)
+          (reference "#PWR0602") (unit 1)
         )
       )
@@
   (symbol (lib_id "SQ2310ES-T1:SQ2310ES-T1") (at 154.94 99.06 0) (unit 1)
     (in_bom yes) (on_board yes) (dnp no) (fields_autoplaced)
-    (property "Reference" "Q1" (at 166.37 95.885 0)
+    (property "Reference" "Q601" (at 166.37 95.885 0)
       (effects (font (size 1.27 1.27)) (justify left))
     )
@@
       (effects (font (size 1.27 1.27)) (justify left))
     )
-    (property "Footprint" "SOT95P237X112-3N" (at 166.37 197.79 0)
+    (property "Footprint" "mod:SOT95P237X112-3N" (at 166.37 197.79 0)
       (effects (font (size 1.27 1.27)) (justify left top) hide)
     )
@@
       (project "Projet_Controler"
         (path "/3b08c5cd-ddb4-4590-8a64-446919e151a7/d5df5f48-8d85-45ba-9c59-31e00cd39d16"
-          (reference "Q1") (unit 1)
+          (reference "Q601") (unit 1)
         )
       )
@@
   (symbol (lib_id "VS-30BQ015HM3_9AT:VS-30BQ015HM3_9AT") (at 154.94 66.04 270) (unit 1)
     (in_bom yes) (on_board yes) (dnp no)
-    (property "Reference" "D1" (at 148.59 73.66 90)
+    (property "Reference" "D601" (at 148.59 73.66 90)
       (effects (font (size 1.27 1.27)) (justify left))
     )
@@
       (effects (font (size 1.27 1.27)) (justify left))
     )
-    (property "Footprint" "DIOM7959X262N" (at 61.29 78.74 0)
+    (property "Footprint" "mod:DIOM7959X262N" (at 61.29 78.74 0)
       (effects (font (size 1.27 1.27)) (justify left top) hide)
     )
@@
       (project "Projet_Controler"
         (path "/3b08c5cd-ddb4-4590-8a64-446919e151a7/d5df5f48-8d85-45ba-9c59-31e00cd39d16"
-          (reference "D1") (unit 1)
-        )
-      )
+          (reference "D601") (unit 1)
+        )
+      )
