File: Hardware/PCB/Projet_Controler V3 - Copie/power.kicad_sch (KiCad schematic)
At the start: 11 parts, among them IC3 LTC4058EDD-4.2#PBF, J1 BATT, J1 USB_B_Micro, U2 BU33SD5WG-TR, U2 WE-TVS-82400102

Commit message: update pcb
Parts:
- removed J1: USB_B_Micro, symbol Connector:USB_B_Micro
- added J302: USB_C_Receptacle_USB2.0, Connector_USB:USB_C_Receptacle_HRO_TYPE-C-31-M-12, symbol Connector:USB_C_Receptacle_USB2.0
- added R302, R303: 5.1k, Resistor_SMD:R_0402_1005Metric, symbol Device:R_Small
- C301: renamed from Cin; footprint (none) -> Capacitor_SMD:C_0402_1005Metric
- C302: renamed from Cout; footprint (none) -> Capacitor_SMD:C_0402_1005Metric
- C303: renamed from C10; footprint (none) -> Capacitor_SMD:C_0402_1005Metric
- C304: renamed from C8; footprint (none) -> Capacitor_SMD:C_0402_1005Metric
- J301: renamed from J1; footprint (none) -> Connector_PinHeader_1.27mm:PinHeader_1x02_P1.27mm_Vertical
- R301: renamed from R12; footprint (none) -> Resistor_SMD:R_0402_1005Metric
- renumbered IC3 to IC301, S1 to S301, U2 to U301, U2 to U302
Connections:
- net +5V: now also J302.A4 (VBUS), J302.A9 (VBUS), J302.B4 (VBUS), J302.B9 (VBUS)
- net GND: now also J302.A1 (GND), J302.A12 (GND), J302.B1 (GND), J302.B12 (GND), J302.S1 (SHIELD), R302.2, R303.1
- net at U302.1: now also J302.A7 (D-), J302.B7 (D-)
- net at U302.3: now also J302.A6 (D+), J302.B6 (D+)
- new net: J302.B5 (CC2), R303.2
- new net: J302.A5 (CC1), R302.1
Other:
- note added: "USB C"
- note removed: "Micro USB type B"
- moved on the sheet: C304, U302
