File: Hardware/PCB/Projet_Controler V3 - Copie/sensors.kicad_sch (KiCad schematic)
At the start: 10 parts, among them IC1 VL53L5CX

Commit message: update pcb
Parts:
- IC401: renamed from IC1; footprint VL53L5CX -> mod:VL53L5CX
- R401: renamed from R9; footprint (none) -> Resistor_SMD:R_0402_1005Metric
- R402: renamed from R10; footprint (none) -> Resistor_SMD:R_0402_1005Metric
- R403: renamed from R5; footprint (none) -> Resistor_SMD:R_0402_1005Metric
- R404: renamed from R4; footprint (none) -> Resistor_SMD:R_0402_1005Metric
- R405: renamed from R8; footprint (none) -> Resistor_SMD:R_0402_1005Metric
- R406: renamed from R11; footprint (none) -> Resistor_SMD:R_0402_1005Metric
- R407: renamed from R1; footprint (none) -> Resistor_SMD:R_0402_1005Metric
- R408: renamed from R3; footprint (none) -> Resistor_SMD:R_0402_1005Metric
- R409: renamed from R2; footprint (none) -> Resistor_SMD:R_0402_1005Metric
