File: Hardware/PCB/Projet_Controler V3 - Copie/stm32.kicad_sch (KiCad schematic)
At the start: 8 parts, among them U1 STM32G431KBTx

Commit message: update pcb
Parts:
- added GND201, NRST201, USART2_RX201, USART2_TX201: TestPoint, TestPoint:TestPoint_Pad_D1.0mm, symbol Connector:TestPoint
- added R201: 10k, Resistor_SMD:R_0402_1005Metric, symbol Device:R_Small
- C201: renamed from C; footprint (none) -> Capacitor_SMD:C_0402_1005Metric
- C202: renamed from C7; footprint (none) -> Capacitor_SMD:C_0402_1005Metric
- C203: renamed from C3; footprint (none) -> Capacitor_SMD:C_0402_1005Metric
- C204: renamed from C2; footprint (none) -> Capacitor_SMD:C_0402_1005Metric
- C205: renamed from C6; footprint (none) -> Capacitor_SMD:C_0402_1005Metric
- SWCLK201: renamed from TP2; footprint TestPoint:TestPoint_Pad_D1.5mm -> TestPoint:TestPoint_Pad_D1.0mm
- SWDIO201: renamed from TP1; footprint TestPoint:TestPoint_Pad_D1.5mm -> TestPoint:TestPoint_Pad_D1.0mm
- renumbered U1 to U201
Connections:
- net +3.3V: no longer U201.31 (PB8)
- net at C201.2, U201.4 (PG10): now also NRST201.1
- net KEY: now reaches U201.5 (PA0)
- net Earth renamed GND
- net GND: now also GND201.1, R201.2
- net TOF_PWR_EN: no longer names the net of U201.12 (PA7)
- net USART2_RX: no longer names the net of U201.7 (PA2)
- net USART2_RX: now also USART2_RX201.1
- net USART2_TX: no longer names the net of U201.8 (PA3)
- net USART2_TX: now also USART2_TX201.1
- new net: R201.1, U201.31 (PB8)
