File: Hardware/PCB/Projet_Controler V4/_autosave-Projet_Controler.kicad_pcb (KiCad board)
At the start: 4 copper layers, 41 x 26 mm, 50 parts, among them IC301 LTC4058EDD-4.2#PBF, IC401 VL53L5CX, J301 BATT, J302 USB_C_Receptacle_USB2.0, J601 MOTOR, Q601 SQ2310ES-T1, U201 STM32G431KBTx, U301 BU33SD5WG-TR, U302 WE-TVS-82400102, U501 HC-05

Commit message: reroutage LF pas assumé à 100%
Routing:
- net /BLUETOOTH/KEY: track 43.1 -> 46.6 mm
- net GND: vias 6 -> 7
Changed lines of the file:
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@@
 			(at 0 -1.448 0)
 			(layer "F.SilkS")
+			(hide yes)
 			(effects
 				(font
@@
 			(at 0 -1.16 0)
 			(layer "F.SilkS")
+			(hide yes)
 			(effects
 				(font
@@
 			(at 0 -5.645 0)
 			(layer "F.SilkS")
+			(hide yes)
 			(effects
 				(font
@@
 			(at 0 -1.695 0)
 			(layer "F.SilkS")
+			(hide yes)
 			(effects
 				(font
@@
 			(at 0 -1.16 90)
 			(layer "F.SilkS")
+			(hide yes)
 			(effects
 				(font
@@
 			(at 0 -2.4 0)
 			(layer "F.SilkS")
+			(hide yes)
 			(effects
 				(font
@@
 			(at 0 -1.17 0)
 			(layer "F.SilkS")
+			(hide yes)
 			(effects
 				(font
@@
 			(at 0 -1.448 0)
 			(layer "F.SilkS")
+			(hide yes)
 			(effects
 				(font
@@
 			(at 0 -1.448 0)
 			(layer "F.SilkS")
+			(hide yes)
 			(effects
 				(font
@@
 			(at 0 -3.35 0)
 			(layer "F.SilkS")
+			(hide yes)
 			(effects
 				(font
@@
 			(at 0 -1.695 90)
 			(layer "F.SilkS")
+			(hide yes)
 			(effects
 				(font
@@
 			(at 0 -1.16 90)
 			(layer "F.SilkS")
+			(hide yes)
 			(effects
 				(font
@@
 			(at 0 -1.17 90)
 			(layer "F.SilkS")
+			(hide yes)
 			(effects
 				(font
@@
 			(at 0 -1.17 90)
 			(layer "F.SilkS")
+			(hide yes)
 			(effects
 				(font
@@
 			(at 0 0.775 0)
 			(layer "F.SilkS")
+			(hide yes)
 			(effects
 				(font
@@
 			(at 0 -1.16 45)
 			(layer "F.SilkS")
+			(hide yes)
 			(effects
 				(font
@@
 			(at 0 -3.35 0)
 			(layer "F.SilkS")
+			(hide yes)
 			(effects
 				(font
@@
 			(at 0 -1.43 90)
 			(layer "F.SilkS")
+			(hide yes)
 			(effects
 				(font
@@
 			(at 0 -5.88 0)
 			(layer "F.SilkS")
+			(hide yes)
 			(effects
 				(font
@@
 			(at 0 -1.16 90)
 			(layer "F.SilkS")
+			(hide yes)
 			(effects
 				(font
@@
 			(at 0 -1.448 0)
 			(layer "F.SilkS")
+			(hide yes)
 			(effects
 				(font
@@
 			(at 0 -1.17 90)
 			(layer "F.SilkS")
+			(hide yes)
 			(effects
 				(font
@@
 			(at 0 -2.45 0)
 			(layer "F.SilkS")
+			(hide yes)
 			(effects
 				(font
@@
 			(at 0 -1.17 90)
 			(layer "F.SilkS")
+			(hide yes)
 			(effects
 				(font
@@
 			(at 0 -1.16 0)
 			(layer "F.SilkS")
+			(hide yes)
 			(effects
 				(font
@@
 			(at 0 -1.16 45)
 			(layer "F.SilkS")
+			(hide yes)
 			(effects
 				(font
@@
 			(at 0 -1.16 90)
 			(layer "F.SilkS")
+			(hide yes)
 			(effects
 				(font
@@
 			(at 0 -1.16 90)
 			(layer "F.SilkS")
+			(hide yes)
 			(effects
 				(font
@@
 			(at 0 -1.43 90)
 			(layer "F.SilkS")
+			(hide yes)
 			(effects
 				(font
@@
 			(at 0 -3.35 0)
 			(layer "F.SilkS")
+			(hide yes)
 			(effects
 				(font
@@
 			(at 0 -1.448 0)
 			(layer "F.SilkS")
+			(hide yes)
 			(effects
 				(font
@@
 			(at 0 -1.17 0)
 			(layer "F.SilkS")
+			(hide yes)
 			(effects
 				(font
@@
 			(at 0 -1.448 0)
 			(layer "F.SilkS")
+			(hide yes)
 			(effects
 				(font
@@
 			(at 0 -3.35 0)
 			(layer "F.SilkS")
+			(hide yes)
 			(effects
 				(font
@@
 			(at 0 1.17 90)
 			(layer "B.SilkS")
+			(hide yes)
 			(effects
 				(font
@@
 			(at 0 1.17 90)
 			(layer "B.SilkS")
+			(hide yes)
 			(effects
 				(font
@@
 			(at 0 1.17 90)
 			(layer "B.SilkS")
+			(hide yes)
 			(effects
 				(font
@@
 			(at 0 1.17 90)
 			(layer "B.SilkS")
+			(hide yes)
 			(effects
 				(font
@@
 			(at 0 1.17 90)
 			(layer "B.SilkS")
+			(hide yes)
 			(effects
 				(font
@@
 			(at 0 1.17 90)
 			(layer "B.SilkS")
+			(hide yes)
 			(effects
 				(font
@@
 			(at 0 1.17 90)
 			(layer "B.SilkS")
+			(hide yes)
 			(effects
 				(font
@@
 			(at 0 0 0)
 			(layer "B.SilkS")
+			(hide yes)
 			(effects
 				(font
@@
 			(at 0 1.17 90)
 			(layer "B.SilkS")
+			(hide yes)
 			(effects
 				(font
@@
 			(at 0 1.17 90)
 			(layer "B.SilkS")
+			(hide yes)
 			(effects
 				(font
@@
 			(at 0 0 90)
 			(layer "B.SilkS")
+			(hide yes)
 			(effects
 				(font
@@
 			(at 0 0 0)
 			(layer "B.SilkS")
+			(hide yes)
 			(effects
 				(font
@@
 			(at 0 2.4 90)
 			(layer "B.SilkS")
+			(hide yes)
 			(effects
 				(font
@@
 			(at 0 1.17 90)
 			(layer "B.SilkS")
+			(hide yes)
 			(effects
 				(font
@@
 			(at 0 1.17 90)
 			(layer "B.SilkS")
+			(hide yes)
 			(effects
 				(font
@@
 	)
 	(via
+		(at 63.7 67.9)
+		(size 0.45)
+		(drill 0.3)
+		(layers "F.Cu" "B.Cu")
+		(free yes)
+		(net 1)
+	)
+	(via
 		(at 48.6 60.2)
 		(size 0.45)
@@
 	)
 	(segment
+		(start 74.3 50.9)
+		(end 70.8 50.9)
+		(width 0.2)
+		(layer "In2.Cu")
+		(net 40)
+	)
+	(segment
 		(start 62.3 54.1)
 		(end 58.8 54.1)
@@
 			)
 		)
+	)
+	(zone
+		(net 0)
+		(net_name "")
+		(layer "B.Cu")
+		(hatch edge 0.5)
+		(connect_pads
+			(clearance 0)
+		)
+		(min_thickness 0.2)
+		(filled_areas_thickness no)
+		(keepout
+			(tracks not_allowed)
+			(vias not_allowed)
+			(pads not_allowed)
+			(copperpour not_allowed)
+			(footprints allowed)
+		)
+		(fill
+			(thermal_gap 0.5)
+			(thermal_bridge_width 0.5)
+		)
+		(polygon
+			(pts
+				(xy 63.8 65.7) (xy 63.8 66.3) (xy 63.3 66.3) (xy 62.9 66) (xy 63.2 65.6)
+			)
+		)
