File: Hardware/PCB/Projet_Controler V4/stm32.kicad_sch (KiCad schematic)
At the start: 13 parts, among them U201 STM32G431KBTx

Commit message: reroutage LF pas assumé à 100%
Parts:
- R201: value 10k -> 100k
Connections:
- net USART2_TX: now reaches U201.8 (PA3), USART2_TX201.1
- net SWDIO: now reaches SWDIO201.1, U201.23 (PA13)
- net NRST: now reaches C201.2, NRST201.1, U201.4 (PG10)
- net BOOT0: now reaches R201.1, U201.31 (PB8)
- net SWCLK: now reaches SWCLK201.1, U201.24 (PA14)
- net USART2_RX: now reaches U201.7 (PA2), USART2_RX201.1
