File: Hardware/PCB/Projet_Controler V5/Projet_Controler.kicad_pcb (KiCad board)
At the start: 4 copper layers, 41 x 26 mm, 50 parts, among them IC301 LTC4058EDD-4.2#PBF, J301 BATT, J302 USB_C_Receptacle_USB2.0, J601 MOTOR, Q601 SQ2310ES-T1, U201 STM32G431KBTx, U301 BU33SD5WG-TR, U302 WE-TVS-82400102, U501 HC-05

Commit message: add gnd via
Routing:
- net +5V: track 24.4 -> 22.6 mm
- net /STM32/USART2_RX: track 14.5 -> 13.0 mm
- net /POWER/BAT: track 32.1 -> 33.2 mm
- net /STM32/USART2_TX: track 19.6 -> 18.8 mm
- net GND: vias 4 -> 14
